Commit message: Modify finder.xacro file to add a laser_link tag Modify finder_rviz.launch file to add gmmaping tag Modify finder_robot.launch file to add the urg_node node

File: catkin_ws/src/hardware/finder_description/urdf/finder.xacro (robot description, xacro)
@@ -268,3 +268,9 @@
       <origin xyz="-0.023 -0.1 0"/>
     </joint>
+	<link name = "laser_link"/>
+<joint name="base_to_laser_joint" type="fixed">
+      <parent link="base_link"/>
+      <child link="laser_link"/>
+      <origin xyz="0.2 0 0.2"/>
+    </joint>
 </robot>
