Commit message: modify the xacro files to change the inertias and gazebo parameters

File: catkin_ws/src/hardware/finder_description/robot/finder_base_4w.gazebo.xacro (robot description, xacro)
@@ -33,8 +33,8 @@
 	<xacro:gazebo_ref link_name="right_back_arm"/>
 	<xacro:gazebo_ref link_name="left_back_arm"/>-->
-  <xacro:gazebo_ref link_name="right_front_wheel_link" kp="100000.0" kd="10.0" mu1="10.5" mu2="10.5" color="White"/>
-  <xacro:gazebo_ref link_name="left_front_wheel_link" kp="100000.0" kd="10.0" mu1="10.5" mu2="10.5" color="White"/>
-  <xacro:gazebo_ref link_name="right_rear_wheel_link" kp="100000.0" kd="10.0" mu1="10.5" mu2="10.5" color="White"/>
-  <xacro:gazebo_ref link_name="left_rear_wheel_link" kp="100000.0" kd="10.0" mu1="10.05" mu2="10.5" color="White"/>
+  <xacro:gazebo_ref link_name="right_front_wheel_link" kp="100000.0" kd="1000.0" mu1="0.5" mu2="2.8" color="White"/>
+  <xacro:gazebo_ref link_name="left_front_wheel_link" kp="100000.0" kd="1000.0" mu1="0.5" mu2="2.8" color="White"/>
+  <xacro:gazebo_ref link_name="right_rear_wheel_link" kp="100000.0" kd="1000.0" mu1="0.5" mu2="2.8" color="White"/>
+  <xacro:gazebo_ref link_name="left_rear_wheel_link" kp="100000.0" kd="1000.0" mu1="0.5" mu2="2.8" color="White"/>
 	<xacro:tran joint="right_front_flipper_joint"/>
 	<xacro:tran joint="left_front_flipper_joint"/>

File: catkin_ws/src/hardware/finder_description/robot/finder_base_4w.urdf.xacro (robot description, xacro)
@@ -70,5 +70,9 @@
 	</link>-->
   <link name="chasis_link">
-    <xacro:inertial_matrix mass="5.0"/>
+    <inertial>
+      <origin xyz="0 0 0" rpy="0 0 0"/>
+      <mass value="5.0"/>
+      <inertia ixx="0.213541666667" ixy="0.0" ixz="0.0" iyy="0.0448955835937" iyz="0.0" izz="0.23968725026"/>
+    </inertial>
     <collision>
       <origin rpy="0 0 0" xyz="0 0 0.155"/>
@@ -86,5 +90,10 @@
   </link>
   <link name="right_front_wheel_link">
-    <xacro:inertial_matrix mass="0.5"/>
+    <!--<xacro:inertial_matrix mass="0.5"/>-->
+    <inertial>
+      <origin xyz="0 0 0" rpy="0 0 0"/>
+      <mass value="0.5"/>
+      <inertia ixx="0.000730417916667" ixy="0.0" ixz="0.0" iyy="0.000730417916667" iyz="0.0" izz="0.0006275025"/>
+    </inertial>
     <collision>
       <origin rpy="0 0 0" xyz="0 0 0"/>
@@ -102,5 +111,10 @@
   </link>
   <link name="left_front_wheel_link">
-    <xacro:inertial_matrix mass="0.5"/>
+    <!--<xacro:inertial_matrix mass="0.5"/>-->
+    <inertial>
+      <origin xyz="0 0 0" rpy="0 0 0"/>
+      <mass value="0.5"/>
+      <inertia ixx="0.000730417916667" ixy="0.0" ixz="0.0" iyy="0.000730417916667" iyz="0.0" izz="0.0006275025"/>
+    </inertial>
     <collision>
       <origin rpy="0 0 0" xyz="0 0 0"/>
@@ -118,5 +132,10 @@
   </link>
   <link name="right_rear_wheel_link">
-    <xacro:inertial_matrix mass="0.5"/>
+    <!--<xacro:inertial_matrix mass="0.5"/>-->
+    <inertial>
+      <origin xyz="0 0 0" rpy="0 0 0"/>
+      <mass value="0.5"/>
+      <inertia ixx="0.000730417916667" ixy="0.0" ixz="0.0" iyy="0.000730417916667" iyz="0.0" izz="0.0006275025"/>
+    </inertial>
     <collision>
       <origin rpy="0 0 0" xyz="0 0 0"/>
@@ -134,5 +153,10 @@
   </link>
   <link name="left_rear_wheel_link">
-    <xacro:inertial_matrix mass="0.5"/>
+    <!--<xacro:inertial_matrix mass="0.5"/>-->
+    <inertial>
+      <origin xyz="0 0 0" rpy="0 0 0"/>
+      <mass value="0.5"/>
+      <inertia ixx="0.000730417916667" ixy="0.0" ixz="0.0" iyy="0.000730417916667" iyz="0.0" izz="0.0006275025"/>
+    </inertial>
     <collision>
       <origin rpy="0 0 0" xyz="0 0 0"/>
@@ -157,5 +181,5 @@
   <parent link = "chasis_link"/>
   <child link = "right_front_wheel_link"/>
-  <origin xyz="-0.1959875 -0.201 0.0501" rpy="0 ${-pi/2} 0"/>
+  <origin xyz="-0.1959875 -0.201 0.0501" rpy="0 ${pi/2} 0"/>
   <axis xyz="0 0 1"/>
 </joint>
@@ -163,5 +187,5 @@
   <parent link = "chasis_link"/>
   <child link = "left_front_wheel_link"/>
-  <origin xyz="0.1959875 -0.201 0.0501" rpy="0 ${-pi/2} 0"/>
+  <origin xyz="0.1959875 -0.201 0.0501" rpy="0 ${pi/2} 0"/>
   <axis xyz="0 0 1"/>
 </joint>
@@ -169,5 +193,5 @@
   <parent link = "chasis_link"/>
   <child link = "right_rear_wheel_link"/>
-  <origin xyz="-0.1959875 0.201 0.0501" rpy="0 ${-pi/2} 0"/>
+  <origin xyz="-0.1959875 0.201 0.0501" rpy="0 ${pi/2} 0"/>
   <axis xyz="0 0 1"/>
 </joint>
@@ -175,5 +199,5 @@
   <parent link = "chasis_link"/>
   <child link = "left_rear_wheel_link"/>
-  <origin xyz="0.1959875 0.201 0.0501" rpy="0 ${-pi/2} 0"/>
+  <origin xyz="0.1959875 0.201 0.0501" rpy="0 ${pi/2} 0"/>
   <axis xyz="0 0 1"/>
 </joint>
