Commit message: add changes to perform mapping

File: catkin_ws/src/hardware/finder_description/robot/finder_base.gazebo.xacro (robot description, xacro)
@@ -36,5 +36,5 @@
 	<xacro:tran joint="right_back_flipper_joint"/>
 	<xacro:tran joint="left_back_flipper_joint"/>
-  <gazebo reference="laser_link">
+  <gazebo reference="base_laser">
     <material>Gazebo/Red</material>
     <sensor type="ray" name="hokuyo_sensor">
@@ -67,5 +67,5 @@
       <plugin name="gazebo_ros_hokuyo_controller" filename="libgazebo_ros_laser.so">
         <topicName>scan</topicName>
-        <frameName>laser_link</frameName> <!-- base_scan -->
+        <frameName>base_laser</frameName> <!-- base_scan -->
       </plugin>
     </sensor>

File: catkin_ws/src/hardware/finder_description/robot/finder_base.urdf.xacro (robot description, xacro)
@@ -93,5 +93,5 @@
 	<!-- brazo trasero izquierdo chasis -->
 	<xacro:lateral_arms name="left_back_arm" cad_name="brazo_der_frontal" origin="0.3264 0.30255 -0.0629"/>
-	<link name = "laser_link">
+	<link name = "base_laser">
 		<visual>
       			<origin xyz="0 0 0.0" rpy="0 0 0"/>
@@ -117,5 +117,5 @@
 	<joint name="base_to_laser_joint" type="fixed">
       		<parent link="base_link"/>
-      		<child link="laser_link"/>
+      		<child link="base_laser"/>
       		<origin xyz="0.4 0 0.27"/>
     	</joint>

File: catkin_ws/src/hardware/finder_description/robot/finder_base_4w.gazebo.xacro (robot description, xacro)
@@ -60,5 +60,5 @@
     </plugin>
   </gazebo>
-  <gazebo reference="laser_link">
+  <gazebo reference="base_laser">
     <material>Gazebo/Red</material>
     <sensor type="ray" name="hokuyo_sensor">
@@ -71,6 +71,6 @@
             <samples>720</samples>
             <resolution>1</resolution>
-            <min_angle>-1.5707</min_angle>
-            <max_angle>1.5707</max_angle>
+            <min_angle>-2.0943</min_angle>
+            <max_angle>2.0943</max_angle>
           </horizontal>
         </scan>
@@ -91,5 +91,5 @@
       <plugin name="gazebo_ros_hokuyo_controller" filename="libgazebo_ros_laser.so">
         <topicName>scan</topicName>
-        <frameName>laser_link</frameName> <!-- base_scan -->
+        <frameName>base_laser</frameName> <!-- base_scan -->
       </plugin>
     </sensor>

File: catkin_ws/src/hardware/finder_description/robot/finder_base_4w.urdf.xacro (robot description, xacro)
@@ -226,5 +226,5 @@
 	<!-- brazo trasero izquierdo chasis -->
 	<xacro:lateral_arms name="left_back_arm" cad_name="brazo_der_frontal" origin="0.3264 0.30255 -0.0629"/>
-	<link name = "laser_link">
+	<link name = "base_laser">
 		<visual>
       			<origin xyz="0 0 0.0" rpy="0 0 0"/>
@@ -250,5 +250,5 @@
 	<joint name="base_to_laser_joint" type="fixed">
       		<parent link="base_link"/>
-      		<child link="laser_link"/>
+      		<child link="base_laser"/>
       		<origin xyz="0.4 0 0.27"/>
     	</joint>

File: catkin_ws/src/hardware/finder_description/robot/finder_base_8w.gazebo.xacro (robot description, xacro)
@@ -33,8 +33,8 @@
 	<xacro:gazebo_ref link_name="right_back_arm"/>
 	<xacro:gazebo_ref link_name="left_back_arm"/>-->
-  <xacro:gazebo_ref link_name="right_front_wheel_link" kp="100000.0" kd="1000.0" mu1="0.5" mu2="2.8" color="orange"/>
-  <xacro:gazebo_ref link_name="left_front_wheel_link" kp="100000.0" kd="1000.0" mu1="0.5" mu2="2.8" color="orange"/>
-  <xacro:gazebo_ref link_name="right_rear_wheel_link" kp="100000.0" kd="1000.0" mu1="0.5" mu2="2.8" color="orange"/>
-  <xacro:gazebo_ref link_name="left_rear_wheel_link" kp="100000.0" kd="1000.0" mu1="0.5" mu2="2.8" color="orange"/>
+  <xacro:gazebo_ref link_name="right_front_wheel_link" kp="100000.0" kd="1000.0" mu1="125" mu2="128" color="orange"/>
+  <xacro:gazebo_ref link_name="left_front_wheel_link" kp="100000.0" kd="1000.0" mu1="125" mu2="128" color="orange"/>
+  <xacro:gazebo_ref link_name="right_rear_wheel_link" kp="100000.0" kd="1000.0" mu1="125" mu2="128" color="orange"/>
+  <xacro:gazebo_ref link_name="left_rear_wheel_link" kp="100000.0" kd="1000.0" mu1="125" mu2="128" color="orange"/>
 <xacro:gazebo_ref link_name="chasis_link" kp="100.0" kd="10.0" mu1="10.0" mu2="10.0" color="grey"/>
 <xacro:gazebo_ref link_name="left_belt_link" kp="100.0" kd="10.0" mu1="10.0" mu2="10.0" color="white"/>
@@ -63,5 +63,5 @@
     </plugin>
   </gazebo>
-  <gazebo reference="laser_link">
+  <gazebo reference="base_laser">
     <material>Gazebo/Red</material>
     <sensor type="ray" name="hokuyo_sensor">
@@ -74,6 +74,6 @@
             <samples>720</samples>
             <resolution>1</resolution>
-            <min_angle>-1.5707</min_angle>
-            <max_angle>1.5707</max_angle>
+            <min_angle>-2.0943</min_angle>
+            <max_angle>2.0943</max_angle>
           </horizontal>
         </scan>
@@ -94,5 +94,5 @@
       <plugin name="gazebo_ros_hokuyo_controller" filename="libgazebo_ros_laser.so">
         <topicName>scan</topicName>
-        <frameName>laser_link</frameName> <!-- base_scan -->
+        <frameName>base_laser</frameName> <!-- base_scan -->
       </plugin>
     </sensor>

File: catkin_ws/src/hardware/finder_description/robot/finder_base_8w.urdf.xacro (robot description, xacro)
@@ -168,4 +168,88 @@
     </visual>
   </link>
+  <link name="right_front_m_wheel_link">
+    <!--<xacro:inertial_matrix mass="0.5"/>-->
+    <inertial>
+      <origin xyz="0 0 0" rpy="0 0 0"/>
+      <mass value="0.5"/>
+      <inertia ixx="0.000730417916667" ixy="0.0" ixz="0.0" iyy="0.000730417916667" iyz="0.0" izz="0.0006275025"/>
+    </inertial>
+    <collision>
+      <origin rpy="0 0 0" xyz="0 0 0"/>
+      <geometry>
+        <cylinder radius="0.0501" length="0.1"/>
+      </geometry>
+    </collision>
+    <visual>
+      <origin rpy="0 0 0" xyz="0 0 0"/>
+      <geometry>
+        <cylinder radius="0.0501" length="0.1"/>
+      </geometry>
+      <material name="white"/>
+    </visual>
+  </link>
+  <link name="left_front_m_wheel_link">
+    <!--<xacro:inertial_matrix mass="0.5"/>-->
+    <inertial>
+      <origin xyz="0 0 0" rpy="0 0 0"/>
+      <mass value="0.5"/>
+      <inertia ixx="0.000730417916667" ixy="0.0" ixz="0.0" iyy="0.000730417916667" iyz="0.0" izz="0.0006275025"/>
+    </inertial>
+    <collision>
+      <origin rpy="0 0 0" xyz="0 0 0"/>
+      <geometry>
+        <cylinder radius="0.0501" length="0.1"/>
+      </geometry>
+    </collision>
+    <visual>
+      <origin rpy="0 0 0" xyz="0 0 0"/>
+      <geometry>
+        <cylinder radius="0.0501" length="0.1"/>
+      </geometry>
+      <material name="white"/>
+    </visual>
+  </link>
+  <link name="right_rear_m_wheel_link">
+    <!--<xacro:inertial_matrix mass="0.5"/>-->
+    <inertial>
+      <origin xyz="0 0 0" rpy="0 0 0"/>
+      <mass value="0.5"/>
+      <inertia ixx="0.000730417916667" ixy="0.0" ixz="0.0" iyy="0.000730417916667" iyz="0.0" izz="0.0006275025"/>
+    </inertial>
+    <collision>
+      <origin rpy="0 0 0" xyz="0 0 0"/>
+      <geometry>
+        <cylinder radius="0.0501" length="0.1"/>
+      </geometry>
+    </collision>
+    <visual>
+      <origin rpy="0 0 0" xyz="0 0 0"/>
+      <geometry>
+        <cylinder radius="0.0501" length="0.1"/>
+      </geometry>
+      <material name="white"/>
+    </visual>
+  </link>
+  <link name="left_rear_m_wheel_link">
+    <!--<xacro:inertial_matrix mass="0.5"/>-->
+    <inertial>
+      <origin xyz="0 0 0" rpy="0 0 0"/>
+      <mass value="0.5"/>
+      <inertia ixx="0.000730417916667" ixy="0.0" ixz="0.0" iyy="0.000730417916667" iyz="0.0" izz="0.0006275025"/>
+    </inertial>
+    <collision>
+      <origin rpy="0 0 0" xyz="0 0 0"/>
+      <geometry>
+        <cylinder radius="0.0501" length="0.1"/>
+      </geometry>
+    </collision>
+    <visual>
+      <origin rpy="0 0 0" xyz="0 0 0"/>
+      <geometry>
+        <cylinder radius="0.0501" length="0.1"/>
+      </geometry>
+      <material name="white"/>
+    </visual>
+  </link>
   <link name = "left_belt_link">
     <inertial>
@@ -206,5 +290,5 @@
   <parent link = "chasis_link"/>
   <child link = "right_front_wheel_link"/>
-  <origin xyz="-0.1959875 -0.201 0.0501" rpy="0 ${pi/2} 0"/>
+  <origin xyz="-0.19575 -0.2005 0.0501" rpy="0 ${pi/2} 0"/>
   <axis xyz="0 0 1"/>
 </joint>
@@ -212,5 +296,5 @@
   <parent link = "chasis_link"/>
   <child link = "left_front_wheel_link"/>
-  <origin xyz="0.1959875 -0.201 0.0501" rpy="0 ${pi/2} 0"/>
+  <origin xyz="0.19575 -0.2005 0.0501" rpy="0 ${pi/2} 0"/>
   <axis xyz="0 0 1"/>
 </joint>
@@ -218,5 +302,5 @@
   <parent link = "chasis_link"/>
   <child link = "right_rear_wheel_link"/>
-  <origin xyz="-0.1959875 0.201 0.0501" rpy="0 ${pi/2} 0"/>
+  <origin xyz="-0.19575 0.2005 0.0501" rpy="0 ${pi/2} 0"/>
   <axis xyz="0 0 1"/>
 </joint>
@@ -224,5 +308,29 @@
   <parent link = "chasis_link"/>
   <child link = "left_rear_wheel_link"/>
-  <origin xyz="0.1959875 0.201 0.0501" rpy="0 ${pi/2} 0"/>
+  <origin xyz="0.19575 0.2005 0.0501" rpy="0 ${pi/2} 0"/>
+  <axis xyz="0 0 1"/>
+</joint>
+<joint name = "right_front_m_wheel_joint" type="continuous">
+  <parent link = "chasis_link"/>
+  <child link = "right_front_m_wheel_link"/>
+  <origin xyz="-0.19575 -0.0675 0.0501" rpy="0 ${pi/2} 0"/>
+  <axis xyz="0 0 1"/>
+</joint>
+<joint name = "left_front_m_wheel_joint" type="continuous">
+  <parent link = "chasis_link"/>
+  <child link = "left_front_m_wheel_link"/>
+  <origin xyz="0.19575 -0.0675 0.0501" rpy="0 ${pi/2} 0"/>
+  <axis xyz="0 0 1"/>
+</joint>
+<joint name = "right_rear_m_wheel_joint" type="continuous">
+  <parent link = "chasis_link"/>
+  <child link = "right_rear_m_wheel_link"/>
+  <origin xyz="-0.19575 0.0675 0.0501" rpy="0 ${pi/2} 0"/>
+  <axis xyz="0 0 1"/>
+</joint>
+<joint name = "left_rear_m_wheel_joint" type="continuous">
+  <parent link = "chasis_link"/>
+  <child link = "left_rear_m_wheel_link"/>
+  <origin xyz="0.19575 0.0675 0.0501" rpy="0 ${pi/2} 0"/>
   <axis xyz="0 0 1"/>
 </joint>
@@ -261,5 +369,5 @@
 	<!-- brazo trasero izquierdo chasis -->
 	<xacro:lateral_arms name="left_back_arm" cad_name="brazo_der_frontal" origin="0.3264 0.30255 -0.0629"/>
-	<link name = "laser_link">
+	<link name = "base_laser">
 		<visual>
       			<origin xyz="0 0 0.0" rpy="0 0 0"/>
@@ -279,5 +387,5 @@
 	<joint name="base_to_laser_joint" type="fixed">
       		<parent link="base_link"/>
-      		<child link="laser_link"/>
+      		<child link="base_laser"/>
       		<origin xyz="0.4 0 0.311"/>
     	</joint>

File: catkin_ws/src/hardware/finder_description/urdf/finder.xacro (robot description, xacro)
@@ -268,8 +268,8 @@
       <origin xyz="-0.023 -0.1 0"/>
     </joint>
-	<link name = "laser_link"/>
+	<link name = "base_laser"/>
 <joint name="base_to_laser_joint" type="fixed">
       <parent link="base_link"/>
-      <child link="laser_link"/>
+      <child link="base_laser"/>
       <origin xyz="0.2 0 0.2"/>
     </joint>
