Commit message: Add colors to the properties file

File: catkin_ws/src/hardware/finder_description/robot/common_properties.xacro (robot description, xacro)
@@ -32,3 +32,9 @@
     <color rgba="1.0 1.0 1.0 1.0"/>
   </material>
+  <material name="pale_goldenrod">
+    <color rgba="${238/255} ${232/255} ${170/255} 1.0"/>
+  </material>
+  <material name="silver">
+    <color rgba="${192/255} ${192/255} ${192/255} 1.0"/>
+  </material>
 </robot>
