Commit message: add xacro tag for the flippers and change the colors

File: catkin_ws/src/hardware/finder_description/robot/finder_base_8w.urdf.xacro (robot description, xacro)
@@ -7,49 +7,72 @@
 NOTA: NO utilizar acentos en codigo ni en comentarios, de lo contrario no se podra convertir a URDF.-->
 <!-- Rojo= X, Verde=Y y Azul= Z (color de los ejes en Rviz)-->
-<robot name="finder_base_8w"  xmlns:xacro="http://www.ros.org/wiki/xacro">
+<robot name="finder_base"  xmlns:xacro="http://www.ros.org/wiki/xacro">
   <xacro:include filename="$(find finder_description)/robot/finder_base_8w.gazebo.xacro"/>
   <xacro:include filename="$(find finder_description)/robot/common_properties.xacro"/>
-	<!-- Macro para "mandar llamar" a las mallas *.obj -->
-	<xacro:macro name="default_geometry" params="cad_dir:=package://finder_description/mallas cad_file extension:=obj">
-        	<geometry>
-		<!-- Typically, STL/DAE/OBJ model units are in mm, but RViz units are in m, hence models must be scaled down by 1000-->
-            		<mesh filename="${cad_dir}/${cad_file}.${extension}" scale="0.001 0.001 0.001"/>
-        	</geometry>
-    	</xacro:macro>
-	<!--General porpuse variables-->
-	<xacro:property name="pi" value = "3.14159265359"/>
-	<!--Inertial matrix macro-->
-   	<xacro:macro name="inertial_matrix" params="mass">
-    		<inertial>
-			<origin xyz="0 0 0" rpy="0 0 0"/>
-      			<mass value="${mass}"/>
-        		<inertia ixx="1.0" ixy="0.0" ixz="0.0" iyy="0.5" iyz="0.0" izz="1.0"/>
-  		</inertial>
-   	</xacro:macro>
-	<!--Macro para crear los eslabones y "mandar llamar" a los brazos laterales del chasis-->
-	<xacro:macro name = "lateral_arms" params="name cad_name origin">
-		<link name = "${name}">
-			<xacro:inertial_matrix mass="0.3"/>
-			<visual>
-				<xacro:default_geometry cad_file = "${cad_name}"/>
-				<origin xyz= "${origin}"/>
-			</visual>
-			<collision>
-				<xacro:default_geometry cad_file = "${cad_name}"/>
-				<origin xyz= "${origin}"/>
-    			</collision>
-		</link>
-	</xacro:macro>
-	<!--Macro para crear las juntas de los brazos laterales con el chasis-->
-	<xacro:macro name = "arms_joints" params="name child origin">
-		<joint name = "${name}" type="revolute">
-			<parent link = "chasis_link"/>
-			<child	link = "${child}"/>
-			<origin xyz ="${origin}"/>
-			<axis xyz = "1 0 0"/>
-			<limit effort="30.0" velocity="0.2" lower="${-pi}" upper="${pi}"/>
-		</joint>
-	</xacro:macro>
-<!--//////////////////////////  base link //////////////////-->
+  <!-- Macro para "mandar llamar" a las mallas *.obj -->
+  <xacro:macro name="default_geometry" params="cad_dir:=package://finder_description/mallas cad_file extension:=obj">
+    <geometry>
+    <!-- Typically, STL/DAE/OBJ model units are in mm, but RViz units are in m, hence models must be scaled down by 1000-->
+      <mesh filename="${cad_dir}/${cad_file}.${extension}" scale="0.001 0.001 0.001"/>
+    </geometry>
+  </xacro:macro>
+  <!--General porpuse variables-->
+  <xacro:property name="pi" value = "3.14159265359"/>
+  <!--Inertial matrix macro-->
+  <xacro:macro name="inertial_matrix" params="mass">
+    <inertial>
+      <origin xyz="0 0 0" rpy="0 0 0"/>
+      <mass value="${mass}"/>
+      <inertia ixx="1.0" ixy="0.0" ixz="0.0" iyy="0.5" iyz="0.0" izz="1.0"/>
+    </inertial>
+  </xacro:macro>
+  <!--Macro para crear los eslabones y "mandar llamar" a los brazos laterales del chasis-->
+  <xacro:macro name = "lateral_arms" params="name cad_name origin">
+    <link name = "${name}">
+      <xacro:inertial_matrix mass="0.3"/>
+      <visual>
+        <xacro:default_geometry cad_file = "${cad_name}"/>
+        <origin xyz= "${origin}"/>
+      </visual>
+      <collision>
+        <xacro:default_geometry cad_file = "${cad_name}"/>
+        <origin xyz= "${origin}"/>
+      </collision>
+    </link>
+  </xacro:macro>
+  <!--Macro para crear las juntas de los brazos laterales con el chasis-->
+  <xacro:macro name = "arms_joints" params="name child origin">
+    <joint name = "${name}" type="revolute">
+      <parent link = "chasis_link"/>
+      <child link = "${child}"/>
+      <origin xyz ="${origin}"/>
+      <axis xyz = "1 0 0"/>
+      <limit effort="30.0" velocity="0.2" lower="${-pi}" upper="${pi}"/>
+    </joint>
+  </xacro:macro>
+  <!-- Macro para crear las ruedas de traccion en simulacion -->
+  <xacro:macro name="wheel_link" params="name">
+  <link name="${name}_wheel_link">
+    <inertial>
+      <origin xyz="0 0 0" rpy="0 0 0"/>
+      <mass value="0.5"/>
+      <inertia ixx="0.000730417916667" ixy="0.0" ixz="0.0" iyy="0.000730417916667" iyz="0.0" izz="0.0006275025"/>
+    </inertial>
+    <collision>
+      <origin rpy="0 0 0" xyz="0 0 0"/>
+      <geometry>
+        <cylinder radius="0.0501" length="0.1"/>
+      </geometry>
+    </collision>
+    <visual>
+      <origin rpy="0 0 0" xyz="0 0 0"/>
+      <geometry>
+        <cylinder radius="0.0501" length="0.1"/>
+      </geometry>
+    <material name="pale_goldenrod"/>
+    </visual>
+  </link>
+  </xacro:macro>
+  <!--//////////////////////////  base link //////////////////-->
   <link name = "base_link"/>
   <link name = "chasis_link">
@@ -58,4 +81,5 @@
       <xacro:default_geometry cad_file="chassis_core" extension="stl"/>
       <origin xyz= "-0.13635 0 0.1556"/>
+      <material name="silver"/>
     </visual>
     <collision>
@@ -64,192 +88,22 @@
     </collision>
   </link>
-<!--  <link name="chasis_link">
-    <inertial>
-      <origin xyz="0 0 0" rpy="0 0 0"/>
-      <mass value="5.0"/>
-      <inertia ixx="0.213541666667" ixy="0.0" ixz="0.0" iyy="0.0448955835937" iyz="0.0" izz="0.23968725026"/>
-    </inertial>
-    <collision>
-      <origin rpy="0 0 0" xyz="0 0 0.155"/>
-      <geometry>
-        <box size="0.291975 0.7 0.15"/>
-      </geometry>
-    </collision>
-    <visual>
-      <origin rpy="0 0 0" xyz="0 0 0.155"/>
-      <geometry>
-        <box size="0.291975 0.7 0.15"/>
-      </geometry>
-    <material name="grey"/>
-    </visual>
-  </link>-->
-  <link name="right_front_wheel_link">
-    <!--<xacro:inertial_matrix mass="0.5"/>-->
-    <inertial>
-      <origin xyz="0 0 0" rpy="0 0 0"/>
-      <mass value="0.5"/>
-      <inertia ixx="0.000730417916667" ixy="0.0" ixz="0.0" iyy="0.000730417916667" iyz="0.0" izz="0.0006275025"/>
-    </inertial>
-    <collision>
-      <origin rpy="0 0 0" xyz="0 0 0"/>
-      <geometry>
-        <cylinder radius="0.0501" length="0.1"/>
-      </geometry>
-    </collision>
-    <visual>
-      <origin rpy="0 0 0" xyz="0 0 0"/>
-      <geometry>
-        <cylinder radius="0.0501" length="0.1"/>
-      </geometry>
-    <material name="white"/>
-    </visual>
-  </link>
-  <link name="left_front_wheel_link">
-    <!--<xacro:inertial_matrix mass="0.5"/>-->
-    <inertial>
-      <origin xyz="0 0 0" rpy="0 0 0"/>
-      <mass value="0.5"/>
-      <inertia ixx="0.000730417916667" ixy="0.0" ixz="0.0" iyy="0.000730417916667" iyz="0.0" izz="0.0006275025"/>
-    </inertial>
-    <collision>
-      <origin rpy="0 0 0" xyz="0 0 0"/>
-      <geometry>
-        <cylinder radius="0.0501" length="0.1"/>
-      </geometry>
-    </collision>
-    <visual>
-      <origin rpy="0 0 0" xyz="0 0 0"/>
-      <geometry>
-        <cylinder radius="0.0501" length="0.1"/>
-      </geometry>
-    <material name="white"/>
-    </visual>
-  </link>
-  <link name="right_rear_wheel_link">
-    <!--<xacro:inertial_matrix mass="0.5"/>-->
-    <inertial>
-      <origin xyz="0 0 0" rpy="0 0 0"/>
-      <mass value="0.5"/>
-      <inertia ixx="0.000730417916667" ixy="0.0" ixz="0.0" iyy="0.000730417916667" iyz="0.0" izz="0.0006275025"/>
-    </inertial>
-    <collision>
-      <origin rpy="0 0 0" xyz="0 0 0"/>
-      <geometry>
-        <cylinder radius="0.0501" length="0.1"/>
-      </geometry>
-    </collision>
-    <visual>
-      <origin rpy="0 0 0" xyz="0 0 0"/>
-      <geometry>
-        <cylinder radius="0.0501" length="0.1"/>
-      </geometry>
-    <material name="white"/>
-    </visual>
-  </link>
-  <link name="left_rear_wheel_link">
-    <!--<xacro:inertial_matrix mass="0.5"/>-->
-    <inertial>
-      <origin xyz="0 0 0" rpy="0 0 0"/>
-      <mass value="0.5"/>
-      <inertia ixx="0.000730417916667" ixy="0.0" ixz="0.0" iyy="0.000730417916667" iyz="0.0" izz="0.0006275025"/>
-    </inertial>
-    <collision>
-      <origin rpy="0 0 0" xyz="0 0 0"/>
-      <geometry>
-        <cylinder radius="0.0501" length="0.1"/>
-      </geometry>
-    </collision>
-    <visual>
-      <origin rpy="0 0 0" xyz="0 0 0"/>
-      <geometry>
-        <cylinder radius="0.0501" length="0.1"/>
-      </geometry>
-    <material name="white"/>
-    </visual>
-  </link>
-  <link name="right_front_m_wheel_link">
-    <!--<xacro:inertial_matrix mass="0.5"/>-->
-    <inertial>
-      <origin xyz="0 0 0" rpy="0 0 0"/>
-      <mass value="0.5"/>
-      <inertia ixx="0.000730417916667" ixy="0.0" ixz="0.0" iyy="0.000730417916667" iyz="0.0" izz="0.0006275025"/>
-    </inertial>
-    <collision>
-      <origin rpy="0 0 0" xyz="0 0 0"/>
-      <geometry>
-        <cylinder radius="0.0501" length="0.1"/>
-      </geometry>
-    </collision>
-    <visual>
-      <origin rpy="0 0 0" xyz="0 0 0"/>
-      <geometry>
-        <cylinder radius="0.0501" length="0.1"/>
-      </geometry>
-      <material name="white"/>
-    </visual>
-  </link>
-  <link name="left_front_m_wheel_link">
-    <!--<xacro:inertial_matrix mass="0.5"/>-->
-    <inertial>
-      <origin xyz="0 0 0" rpy="0 0 0"/>
-      <mass value="0.5"/>
-      <inertia ixx="0.000730417916667" ixy="0.0" ixz="0.0" iyy="0.000730417916667" iyz="0.0" izz="0.0006275025"/>
-    </inertial>
-    <collision>
-      <origin rpy="0 0 0" xyz="0 0 0"/>
-      <geometry>
-        <cylinder radius="0.0501" length="0.1"/>
-      </geometry>
-    </collision>
-    <visual>
-      <origin rpy="0 0 0" xyz="0 0 0"/>
-      <geometry>
-        <cylinder radius="0.0501" length="0.1"/>
-      </geometry>
-      <material name="white"/>
-    </visual>
-  </link>
-  <link name="right_rear_m_wheel_link">
-    <!--<xacro:inertial_matrix mass="0.5"/>-->
-    <inertial>
-      <origin xyz="0 0 0" rpy="0 0 0"/>
-      <mass value="0.5"/>
-      <inertia ixx="0.000730417916667" ixy="0.0" ixz="0.0" iyy="0.000730417916667" iyz="0.0" izz="0.0006275025"/>
-    </inertial>
-    <collision>
-      <origin rpy="0 0 0" xyz="0 0 0"/>
-      <geometry>
-        <cylinder radius="0.0501" length="0.1"/>
-      </geometry>
-    </collision>
-    <visual>
-      <origin rpy="0 0 0" xyz="0 0 0"/>
-      <geometry>
-        <cylinder radius="0.0501" length="0.1"/>
-      </geometry>
-      <material name="white"/>
-    </visual>
-  </link>
-  <link name="left_rear_m_wheel_link">
-    <!--<xacro:inertial_matrix mass="0.5"/>-->
-    <inertial>
-      <origin xyz="0 0 0" rpy="0 0 0"/>
-      <mass value="0.5"/>
-      <inertia ixx="0.000730417916667" ixy="0.0" ixz="0.0" iyy="0.000730417916667" iyz="0.0" izz="0.0006275025"/>
-    </inertial>
-    <collision>
-      <origin rpy="0 0 0" xyz="0 0 0"/>
-      <geometry>
-        <cylinder radius="0.0501" length="0.1"/>
-      </geometry>
-    </collision>
-    <visual>
-      <origin rpy="0 0 0" xyz="0 0 0"/>
-      <geometry>
-        <cylinder radius="0.0501" length="0.1"/>
-      </geometry>
-      <material name="white"/>
-    </visual>
-  </link>
+  <!--////////////// brazos laterales del chasis ////////////////////-->
+  <!-- brazo frontal derecho chasis -->
+  <xacro:lateral_arms name="right_front_arm" cad_name="brazo_der_frontal" origin="0.3264 0.30255 -0.0629"/>
+  <!-- brazo frontal izquierdo chasis -->
+  <xacro:lateral_arms name="left_front_arm" cad_name="brazo_der_frontal" origin="0.3264 0.30255 -0.0629"/>
+  <!-- brazo trasero derecho chasis -->
+  <xacro:lateral_arms name="right_back_arm" cad_name="brazo_der_frontal" origin="0.3264 0.30255 -0.0629"/>
+  <!-- brazo trasero izquierdo chasis -->
+  <xacro:lateral_arms name="left_back_arm" cad_name="brazo_der_frontal" origin="0.3264 0.30255 -0.0629"/>
+  <!-- ruedas para traccion skid-steer en la simulacion -->
+  <xacro:wheel_link name="right_front"/>
+  <xacro:wheel_link name="left_front"/>
+  <xacro:wheel_link name="right_rear"/>
+  <xacro:wheel_link name="left_rear"/>
+  <xacro:wheel_link name="right_front_m"/>
+  <xacro:wheel_link name="left_front_m"/>
+  <xacro:wheel_link name="right_rear_m"/>
+  <xacro:wheel_link name="left_rear_m"/>
   <link name = "left_belt_link">
     <inertial>
@@ -261,4 +115,5 @@
       <xacro:default_geometry cad_file="belt" extension="stl"/>
       <origin xyz= "0 0 0"/>
+      <material name="white"/>
     </visual>
     <!--<collision>
@@ -276,4 +131,5 @@
       <xacro:default_geometry cad_file="belt" extension="stl"/>
       <origin xyz= "0 0 0"/>
+      <material name="white"/>
     </visual>
     <!--<collision>
@@ -282,9 +138,47 @@
     </collision>-->
   </link>
-<joint name = "chasis_adjustment_joint" type="fixed">
-  <parent link = "base_link"/>
-  <child link = "chasis_link"/>
-  <origin xyz="0 0 0" rpy="0 0 ${pi/2}"/>
-</joint>
+  <link name = "base_laser">
+    <visual>
+      <origin xyz="0 0 0.0" rpy="0 0 0"/>
+      <geometry>
+        <box size="0.01 0.01 0.01"/>
+      </geometry>
+      <material name="red"/>
+    </visual>
+    <inertial>
+      <mass value="0.114" />
+      <origin xyz="0 0 0" />
+      <inertia ixx="0.001" ixy="0.0" ixz="0.0" iyy="0.001" iyz="0.0" izz="0.001" />
+    </inertial>
+  </link>
+  <link name="camera1_link">
+    <visual>
+      <origin xyz="0 0 0" rpy="0 0 0"/>
+      <geometry>
+        <box size="0.01 0.01 0.01"/>
+      </geometry>
+      <material name="red"/>
+    <inertial>
+      <mass value="0.05" />
+      <origin xyz="0 0 0" />
+      <inertia ixx="0.001" ixy="0.0" ixz="0.0" iyy="0.001" iyz="0.0" izz="0.001" />
+    </inertial>
+    </visual>
+  </link>
+  <!--Esta transformacion se hace para que los datos del SLAM correspondan a la correcta orientacion del robot-->
+  <joint name = "chasis_adjustment_joint" type="fixed">
+    <parent link = "base_link"/>
+    <child link = "chasis_link"/>
+    <origin xyz="0 0 0" rpy="0 0 ${pi/2}"/>
+  </joint>
+<!--////////////////// juntas de los brazos laterales del chasis //////////////////-->
+  <!-- junta del brazo frontal derecho -->
+  <xacro:arms_joints name="right_front_flipper_joint" child="right_front_arm" origin="-0.3264 -0.30255 0.1556"/>
+  <!-- junta del brazo frontal izquierdo -->
+  <xacro:arms_joints name="left_front_flipper_joint" child="left_front_arm" origin="0.3264 -0.30255 0.1556"/>
+  <!-- junta del brazo trasero derecho -->
+  <xacro:arms_joints name="right_back_flipper_joint" child="right_back_arm" origin="-0.3264 0.30255 0.1556"/>
+  <!-- junta del brazo trasero izquierdo -->
+  <xacro:arms_joints name="left_back_flipper_joint" child="left_back_arm" origin="0.3264 0.30255 0.1556"/>
 <joint name = "right_front_wheel_joint" type="continuous">
   <parent link = "chasis_link"/>
@@ -329,64 +223,29 @@
   <axis xyz="0 0 1"/>
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