Commit message: Add colors and properties to the flippers

File: catkin_ws/src/hardware/finder_description/robot/finder_base_8w.gazebo.xacro (robot description, xacro)
@@ -1,49 +1,57 @@
 <?xml version="1.0"?>
-<robot name="finder_base_4w_sim" xmlns:xacro="http://ros.org/wiki/xacro">
-    <xacro:arg name="laser_visual" default="true"/>
-	<!-- gazebo tag macro -->
-	<xacro:macro name="gazebo_ref" params="link_name kp kd mu1 mu2 color">
-		<gazebo reference="${link_name}">
-			<kp>${kp}</kp>	<!-- static contact stifness -->
-			<kd>${kd}</kd>	<!-- dynamic contact stifness -->
-			<mu1>${mu1}</mu1>	<!-- static friction coeficient -->
-			<mu2>${mu2}</mu2>	<!-- dynamic friction coeficient -->
-			<material>Gazebo/${color}</material>
-		</gazebo>
-	</xacro:macro>
-	<xacro:macro name="tran" params="joint">
-    		<transmission name="${joint}_tran">
-        		<type>transmission_interface/SimpleTransmission</type>
-        		<joint name="${joint}">
-            			<hardwareInterface>hardware_interface/EffortJointInterface</hardwareInterface>
-        		</joint>
-       			<actuator name="${joint}_motor">
-            			<hardwareInterface>hardware_interface/EffortJointInterface</hardwareInterface>
-           			<mechanicalReduction>1</mechanicalReduction>
-        		</actuator>
-    		</transmission>
-	</xacro:macro>
-	<gazebo>
-        	<plugin name="gazebo_ros_control" filename="libgazebo_ros_control.so">
-			<robotNamespace>/finder_base</robotNamespace>
-        	</plugin>
-    	</gazebo>
-	<!--<xacro:gazebo_ref link_name="right_front_arm" kp="1000.0" kd="1000.0" mu1="10.0" mu2="10.0" color="White"/>
-	<xacro:gazebo_ref link_name="left_front_arm"/>
-	<xacro:gazebo_ref link_name="right_back_arm"/>
-	<xacro:gazebo_ref link_name="left_back_arm"/>-->
-  <xacro:gazebo_ref link_name="right_front_wheel_link" kp="100000.0" kd="1000.0" mu1="125" mu2="128" color="orange"/>
-  <xacro:gazebo_ref link_name="left_front_wheel_link" kp="100000.0" kd="1000.0" mu1="125" mu2="128" color="orange"/>
-  <xacro:gazebo_ref link_name="right_rear_wheel_link" kp="100000.0" kd="1000.0" mu1="125" mu2="128" color="orange"/>
-  <xacro:gazebo_ref link_name="left_rear_wheel_link" kp="100000.0" kd="1000.0" mu1="125" mu2="128" color="orange"/>
-<xacro:gazebo_ref link_name="chasis_link" kp="100.0" kd="10.0" mu1="10.0" mu2="10.0" color="grey"/>
-<xacro:gazebo_ref link_name="left_belt_link" kp="100.0" kd="10.0" mu1="10.0" mu2="10.0" color="white"/>
-<xacro:gazebo_ref link_name="right_belt_link" kp="100.0" kd="10.0" mu1="10.0" mu2="10.0" color="white"/>
-	<xacro:tran joint="right_front_flipper_joint"/>
-	<xacro:tran joint="left_front_flipper_joint"/>
-	<xacro:tran joint="right_back_flipper_joint"/>
-	<xacro:tran joint="left_back_flipper_joint"/>
+<robot name="finder_base" xmlns:xacro="http://ros.org/wiki/xacro">
+  <xacro:arg name="laser_visual" default="true"/>
+  <!-- gazebo tag macro -->
+  <xacro:macro name="gazebo_ref" params="link_name kp kd mu1 mu2 color">
+    <gazebo reference="${link_name}">
+	<kp>${kp}</kp>	<!-- static contact stifness -->
+	<kd>${kd}</kd>	<!-- dynamic contact stifness -->
+	<mu1>${mu1}</mu1>	<!-- static friction coeficient -->
+	<mu2>${mu2}</mu2>	<!-- dynamic friction coeficient -->
+	<material>Gazebo/${color}</material>
+    </gazebo>
+  </xacro:macro>
+  <xacro:macro name="tran" params="joint">
+    <transmission name="${joint}_tran">
+      <type>transmission_interface/SimpleTransmission</type>
+      <joint name="${joint}">
+        <hardwareInterface>hardware_interface/EffortJointInterface</hardwareInterface>
+      </joint>
+      <actuator name="${joint}_motor">
+        <hardwareInterface>hardware_interface/EffortJointInterface</hardwareInterface>
+        <mechanicalReduction>1</mechanicalReduction>
+      </actuator>
+    </transmission>
+  </xacro:macro>
+  <gazebo>
+    <plugin name="gazebo_ros_control" filename="libgazebo_ros_control.so">
+      <robotNamespace>/finder_base</robotNamespace>
+    </plugin>
+  </gazebo>
+  <xacro:gazebo_ref link_name="right_front_arm" kp="1000.0" kd="1000.0" mu1="10.0" mu2="10.0" color="White"/>
+  <xacro:gazebo_ref link_name="left_front_arm" kp="1000.0" kd="1000.0" mu1="10.0" mu2="10.0" color="White"/>
+  <xacro:gazebo_ref link_name="right_back_arm" kp="1000.0" kd="1000.0" mu1="10.0" mu2="10.0" color="White"/>
+  <xacro:gazebo_ref link_name="left_back_arm" kp="1000.0" kd="1000.0" mu1="10.0" mu2="10.0" color="White"/>
+  <xacro:gazebo_ref link_name="right_front_wheel_link" kp="100000.0" kd="1000.0" mu1="100" mu2="100" color="ZincYellow"/>
+  <xacro:gazebo_ref link_name="left_front_wheel_link" kp="100000.0" kd="1000.0" mu1="100" mu2="100" color="ZincYellow"/>
+  <xacro:gazebo_ref link_name="right_rear_wheel_link" kp="100000.0" kd="1000.0" mu1="100" mu2="100" color="ZincYellow"/>
+  <xacro:gazebo_ref link_name="left_rear_wheel_link" kp="100000.0" kd="1000.0" mu1="100" mu2="100" color="ZincYellow"/>
+  <xacro:gazebo_ref link_name="right_front_m_wheel_link" kp="100000.0" kd="1000.0" mu1="100" mu2="100" color="ZincYellow"/>
+  <xacro:gazebo_ref link_name="left_front_m_wheel_link" kp="100000.0" kd="1000.0" mu1="100" mu2="100" color="ZincYellow"/>
+  <xacro:gazebo_ref link_name="right_rear_m_wheel_link" kp="100000.0" kd="1000.0" mu1="100" mu2="100" color="ZincYellow"/>
+  <xacro:gazebo_ref link_name="left_rear_m_wheel_link" kp="100000.0" kd="1000.0" mu1="100" mu2="100" color="ZincYellow"/>
+  <xacro:gazebo_ref link_name="chasis_link" kp="100.0" kd="10.0" mu1="10.0" mu2="10.0" color="Grey"/>
+  <xacro:gazebo_ref link_name="left_belt_link" kp="100.0" kd="10.0" mu1="10.0" mu2="10.0" color="White"/>
+  <xacro:gazebo_ref link_name="right_belt_link" kp="100.0" kd="10.0" mu1="10.0" mu2="10.0" color="White"/>
+  <xacro:tran joint="right_front_flipper_joint"/>
+  <xacro:tran joint="left_front_flipper_joint"/>
+  <xacro:tran joint="right_back_flipper_joint"/>
+  <xacro:tran joint="left_back_flipper_joint"/>
   <gazebo>
     <plugin name="skid_steer_drive_controller" filename="libgazebo_ros_skid_steer_drive.so">
+      <commandTopic>cmd_vel</commandTopic>
+      <odometryTopic>odom</odometryTopic>
+      <odometryFrame>odom</odometryFrame>
+      <robotBaseFrame>base_link</robotBaseFrame>
       <updateRate>25.0</updateRate>
       <robotNamespace>/</robotNamespace>
@@ -52,13 +60,35 @@
       <leftRearJoint>left_rear_wheel_joint</leftRearJoint>
       <rightRearJoint>right_rear_wheel_joint</rightRearJoint>
-      <wheelSeparation>0.401</wheelSeparation>
+      <wheelSeparation>0.3915</wheelSeparation>
       <wheelDiameter>0.1002</wheelDiameter>
-      <robotBaseFrame>base_link</robotBaseFrame>
       <torque>20</torque>
-      <topicName>cmd_vel</topicName>
+      <broadcastTF>true</broadcastTF>
+    </plugin>
+  </gazebo>
+<!-- second controller for the 4 middle-wheels -->
+  <gazebo>
+    <plugin name="skid_steer_drive_controller_2" filename="libgazebo_ros_skid_steer_drive.so">
       <commandTopic>cmd_vel</commandTopic>
       <odometryTopic>odom</odometryTopic>
       <odometryFrame>odom</odometryFrame>
-      <broadcastTF>1</broadcastTF>
+      <robotBaseFrame>base_link</robotBaseFrame>
+      <updateRate>25.0</updateRate>
+      <robotNamespace>/</robotNamespace>
+      <leftFrontJoint>left_front_m_wheel_joint</leftFrontJoint>
+      <rightFrontJoint>right_front_m_wheel_joint</rightFrontJoint>
+      <leftRearJoint>left_rear_m_wheel_joint</leftRearJoint>
+      <rightRearJoint>right_rear_m_wheel_joint</rightRearJoint>
+      <wheelSeparation>0.3915</wheelSeparation>
+      <wheelDiameter>0.1002</wheelDiameter>
+      <torque>20</torque>
+      <broadcastTF>true</broadcastTF>
+    </plugin>
+  </gazebo>
+<!-- plug-in for publish the joint states of the 8 wheels -->
+  <gazebo>
+    <plugin name="joint_state_publisher" filename="libgazebo_ros_joint_state_publisher.so">
+      <jointName>left_front_wheel_joint, right_front_wheel_joint, left_rear_wheel_joint, right_rear_wheel_joint, left_front_m_wheel_joint, right_front_m_wheel_joint, left_rear_m_wheel_joint, right_rear_m_wheel_joint</jointName>
+      <robotNamespace>/finder_base</robotNamespace>
+      <updateRate>25.0</updateRate>
     </plugin>
   </gazebo>
@@ -72,13 +102,13 @@
         <scan>
           <horizontal>
-            <samples>720</samples>
-            <resolution>1</resolution>
-            <min_angle>-2.0943</min_angle>
-            <max_angle>2.0943</max_angle>
+            <samples>240</samples> <!-- with 360deg/1024steps, 240degrees are 682 steps -->
+            <resolution>1.0</resolution> <!-- 0.352 degree, 360deg/1024 steps -->
+            <min_angle>-2.094395</min_angle> <!-- -120 degrees -->
+            <max_angle>2.094395</max_angle>
           </horizontal>
         </scan>
         <range>
-          <min>0.120</min>
-          <max>3.5</max>
+          <min>0.10</min>
+          <max>5.6</max>
           <resolution>0.015</resolution>
         </range>
@@ -98,3 +128,44 @@
     </sensor>
   </gazebo>
+  <!-- tag for simulating the camera1 -->
+  <gazebo reference="camera1_link">
+    <sensor type="camera" name="camera1">
+      <update_rate>30.0</update_rate>
+      <camera name="head">
+          <pose>0 0 0 0 0.5 0</pose>
+        <horizontal_fov>1.3962634</horizontal_fov>
+        <image>
+          <width>400</width>
+          <height>400</height>
+          <format>R8G8B8</format>
+        </image>
+        <clip>
+          <near>0.02</near>
+          <far>300</far>
+        </clip>
+        <noise>
+          <type>gaussian</type>
+          <!-- Noise is sampled independently per pixel on each frame.
+               That pixel's noise value is added to each of its color
+               channels, which at that point lie in the range [0,1]. -->
+          <mean>0.0</mean>
+          <stddev>0.007</stddev>
+        </noise>
+      </camera>
+      <plugin name="camera_controller" filename="libgazebo_ros_camera.so">
+        <alwaysOn>true</alwaysOn>
+        <updateRate>0.0</updateRate>
+        <cameraName>finder_base/camera1</cameraName>
+        <imageTopicName>image_raw</imageTopicName>
+        <cameraInfoTopicName>camera_info</cameraInfoTopicName>
+        <frameName>camera1_link</frameName>
+        <hackBaseline>0.07</hackBaseline>
+        <distortionK1>0.0</distortionK1>
+        <distortionK2>0.0</distortionK2>
+        <distortionK3>0.0</distortionK3>
+        <distortionT1>0.0</distortionT1>
+        <distortionT2>0.0</distortionT2>
+      </plugin>
+    </sensor>
+  </gazebo>
 </robot>

Commit message: change to base_link instead of chasis_link and add base_footprint, add the IMU tag to simulate

File: catkin_ws/src/hardware/finder_description/robot/finder_base_8w.gazebo.xacro (robot description, xacro)
@@ -2,4 +2,5 @@
 <robot name="finder_base" xmlns:xacro="http://ros.org/wiki/xacro">
   <xacro:arg name="laser_visual" default="true"/>
+  <xacro:arg name="imu_visual"   default="false"/>
   <!-- gazebo tag macro -->
   <xacro:macro name="gazebo_ref" params="link_name kp kd mu1 mu2 color">
@@ -41,5 +42,5 @@
   <xacro:gazebo_ref link_name="right_rear_m_wheel_link" kp="100000.0" kd="1000.0" mu1="100" mu2="100" color="ZincYellow"/>
   <xacro:gazebo_ref link_name="left_rear_m_wheel_link" kp="100000.0" kd="1000.0" mu1="100" mu2="100" color="ZincYellow"/>
-  <xacro:gazebo_ref link_name="chasis_link" kp="100.0" kd="10.0" mu1="10.0" mu2="10.0" color="Grey"/>
+  <xacro:gazebo_ref link_name="base_link" kp="100.0" kd="10.0" mu1="10.0" mu2="10.0" color="Grey"/>
   <xacro:gazebo_ref link_name="left_belt_link" kp="100.0" kd="10.0" mu1="10.0" mu2="10.0" color="White"/>
   <xacro:gazebo_ref link_name="right_belt_link" kp="100.0" kd="10.0" mu1="10.0" mu2="10.0" color="White"/>
@@ -53,5 +54,5 @@
       <odometryTopic>odom</odometryTopic>
       <odometryFrame>odom</odometryFrame>
-      <robotBaseFrame>base_link</robotBaseFrame>
+      <robotBaseFrame>base_footprint</robotBaseFrame>
       <updateRate>25.0</updateRate>
       <robotNamespace>/</robotNamespace>
@@ -72,5 +73,5 @@
       <odometryTopic>odom</odometryTopic>
       <odometryFrame>odom</odometryFrame>
-      <robotBaseFrame>base_link</robotBaseFrame>
+      <robotBaseFrame>base_footprint</robotBaseFrame>
       <updateRate>25.0</updateRate>
       <robotNamespace>/</robotNamespace>
@@ -169,3 +170,39 @@
     </sensor>
   </gazebo>
+  <gazebo reference="imu_link">
+    <sensor type="imu" name="imu">
+      <always_on>true</always_on>
+      <visualize>$(arg imu_visual)</visualize>
+    </sensor>
+    <material>Gazebo/FlatBlack</material>
+  </gazebo>
+  <!-- imu plug in -->
+  <gazebo>
+    <plugin name="imu_plugin" filename="libgazebo_ros_imu.so">
+      <alwaysOn>true</alwaysOn>
+      <bodyName>imu_link</bodyName>
+      <frameName>imu_link</frameName>
+      <topicName>imu</topicName>
+      <serviceName>imu_service</serviceName>
+      <gaussianNoise>0.0</gaussianNoise>
+      <updateRate>200</updateRate>
+      <imu>
+        <noise>
+          <type>gaussian</type>
+          <rate>
+            <mean>0.0</mean>
+            <stddev>2e-4</stddev>
+            <bias_mean>0.0000075</bias_mean>
+            <bias_stddev>0.0000008</bias_stddev>
+          </rate>
+          <accel>
+            <mean>0.0</mean>
+            <stddev>1.7e-2</stddev>
+            <bias_mean>0.1</bias_mean>
+            <bias_stddev>0.001</bias_stddev>
+          </accel>
+        </noise>
+      </imu>
+    </plugin>
+  </gazebo>
 </robot>

File: catkin_ws/src/hardware/finder_description/robot/finder_base_8w.urdf.xacro (robot description, xacro)
@@ -44,7 +44,7 @@
   <xacro:macro name = "arms_joints" params="name child origin">
     <joint name = "${name}" type="revolute">
-      <parent link = "chasis_link"/>
+      <parent link = "base_link"/>
       <child link = "${child}"/>
-      <origin xyz ="${origin}"/>
+      <origin xyz ="${origin}" rpy="0 0 ${pi/2}"/>
       <axis xyz = "1 0 0"/>
       <limit effort="30.0" velocity="0.2" lower="${-pi}" upper="${pi}"/>
@@ -75,15 +75,15 @@
   </xacro:macro>
   <!--//////////////////////////  base link //////////////////-->
-  <link name = "base_link"/>
-  <link name = "chasis_link">
+  <link name = "base_footprint"/>
+  <link name = "base_link">
     <xacro:inertial_matrix mass="5.0"/>
     <visual>
       <xacro:default_geometry cad_file="chassis_core" extension="stl"/>
-      <origin xyz= "-0.13635 0 0.1556"/>
+      <origin xyz= "0 -0.13635 0.0707856" rpy="0 0 ${pi/2}"/>
       <material name="silver"/>
     </visual>
     <collision>
       <xacro:default_geometry cad_file="chassis_core" extension="stl"/>
-      <origin xyz= "-0.13635 0 0.1556"/>
+      <origin xyz= "0 -0.13635 0.0707856" rpy="0 0 ${pi/2}"/>
     </collision>
   </link>
@@ -166,81 +166,82 @@
     </visual>
   </link>
+  <link name="imu_link"/>
   <!--Esta transformacion se hace para que los datos del SLAM correspondan a la correcta orientacion del robot-->
-  <joint name = "chasis_adjustment_joint" type="fixed">
-    <parent link = "base_link"/>
-    <child link = "chasis_link"/>
-    <origin xyz="0 0 0" rpy="0 0 ${pi/2}"/>
+  <joint name = "base_joint" type="fixed">
+    <parent link = "base_footprint"/>
+    <child link = "base_link"/>
+    <origin xyz="0 0 0.0848144" rpy="0 0 0"/>
   </joint>
 <!--////////////////// juntas de los brazos laterales del chasis //////////////////-->
   <!-- junta del brazo frontal derecho -->
-  <xacro:arms_joints name="right_front_flipper_joint" child="right_front_arm" origin="-0.3264 -0.30255 0.1556"/>
+  <xacro:arms_joints name="right_front_flipper_joint" child="right_front_arm" origin=" 0.30255 -0.3264 0.0707856"/>
   <!-- junta del brazo frontal izquierdo -->
-  <xacro:arms_joints name="left_front_flipper_joint" child="left_front_arm" origin="0.3264 -0.30255 0.1556"/>
+  <xacro:arms_joints name="left_front_flipper_joint" child="left_front_arm" origin=" 0.30255 0.3264 0.0707856"/>
   <!-- junta del brazo trasero derecho -->
-  <xacro:arms_joints name="right_back_flipper_joint" child="right_back_arm" origin="-0.3264 0.30255 0.1556"/>
+  <xacro:arms_joints name="right_back_flipper_joint" child="right_back_arm" origin="-0.30255 -0.3264 0.0707856"/>
   <!-- junta del brazo trasero izquierdo -->
-  <xacro:arms_joints name="left_back_flipper_joint" child="left_back_arm" origin="0.3264 0.30255 0.1556"/>
+  <xacro:arms_joints name="left_back_flipper_joint" child="left_back_arm" origin="-0.30255 0.3264 0.0707856"/>
 <joint name = "right_front_wheel_joint" type="continuous">
-  <parent link = "chasis_link"/>
+  <parent link = "base_link"/>
   <child link = "right_front_wheel_link"/>
-  <origin xyz="-0.19575 -0.2005 0.0501" rpy="0 ${pi/2} 0"/>
+  <origin xyz="0.2005 -0.19575 -0.0347144" rpy="${-pi/2} 0 0"/>
   <axis xyz="0 0 1"/>
 </joint>
 <joint name = "left_front_wheel_joint" type="continuous">
-  <parent link = "chasis_link"/>
+  <parent link = "base_link"/>
   <child link = "left_front_wheel_link"/>
-  <origin xyz="0.19575 -0.2005 0.0501" rpy="0 ${pi/2} 0"/>
+  <origin xyz="0.2005 0.19575 -0.0347144" rpy="${-pi/2} 0 0"/>
   <axis xyz="0 0 1"/>
 </joint>
 <joint name = "right_rear_wheel_joint" type="continuous">
-  <parent link = "chasis_link"/>
+  <parent link = "base_link"/>
   <child link = "right_rear_wheel_link"/>
-  <origin xyz="-0.19575 0.2005 0.0501" rpy="0 ${pi/2} 0"/>
+  <origin xyz="-0.2005 -0.19575 -0.0347144" rpy="${-pi/2} 0 0"/>
   <axis xyz="0 0 1"/>
 </joint>
 <joint name = "left_rear_wheel_joint" type="continuous">
-  <parent link = "chasis_link"/>
+  <parent link = "base_link"/>
   <child link = "left_rear_wheel_link"/>
-  <origin xyz="0.19575 0.2005 0.0501" rpy="0 ${pi/2} 0"/>
+  <origin xyz="-0.2005 0.19575 -0.0347144" rpy="${-pi/2} 0 0"/>
   <axis xyz="0 0 1"/>
 </joint>
 <joint name = "right_front_m_wheel_joint" type="continuous">
-  <parent link = "chasis_link"/>
+  <parent link = "base_link"/>
   <child link = "right_front_m_wheel_link"/>
-  <origin xyz="-0.19575 -0.0675 0.0501" rpy="0 ${pi/2} 0"/>
+  <origin xyz="0.0675 -0.19575 -0.0347144" rpy="${-pi/2} 0 0"/>
   <axis xyz="0 0 1"/>
 </joint>
 <joint name = "left_front_m_wheel_joint" type="continuous">
-  <parent link = "chasis_link"/>
+  <parent link = "base_link"/>
   <child link = "left_front_m_wheel_link"/>
-  <origin xyz="0.19575 -0.0675 0.0501" rpy="0 ${pi/2} 0"/>
+  <origin xyz="0.0675 0.19575 -0.0347144" rpy="${-pi/2} 0 0"/>
   <axis xyz="0 0 1"/>
 </joint>
 <joint name = "right_rear_m_wheel_joint" type="continuous">
-  <parent link = "chasis_link"/>
+  <parent link = "base_link"/>
   <child link = "right_rear_m_wheel_link"/>
-  <origin xyz="-0.19575 0.0675 0.0501" rpy="0 ${pi/2} 0"/>
+  <origin xyz="-0.0675 -0.19575 -0.0347144" rpy="${-pi/2} 0 0"/>
   <axis xyz="0 0 1"/>
 </joint>
   <joint name = "left_rear_m_wheel_joint" type="continuous">
-    <parent link = "chasis_link"/>
+    <parent link = "base_link"/>
     <child link = "left_rear_m_wheel_link"/>
-    <origin xyz="0.19575 0.0675 0.0501" rpy="0 ${pi/2} 0"/>
+    <origin xyz="-0.0675 0.19575 -0.0347144" rpy="${-pi/2} 0 0"/>
     <axis xyz="0 0 1"/>
   </joint>
   <joint name = "chassis_left_belt_joint" type="fixed">
-    <parent link = "chasis_link"/>
+    <parent link = "base_link"/>
     <child link = "left_belt_link"/>
-    <origin xyz="0.19575 -0.3025 0.1556" rpy="0 0 ${pi/2}"/>
+    <origin xyz="-0.3025 0.19575 0.0707856" rpy="0 0 0"/>
   </joint>
   <joint name = "chassis_right_belt_joint" type="fixed">
-    <parent link = "chasis_link"/>
+    <parent link = "base_link"/>
     <child link = "right_belt_link"/>
-    <origin xyz="-0.19575 -0.3025 0.1556" rpy="0 0 ${pi/2}"/>
+    <origin xyz="-0.3025 -0.19575 0.0707856" rpy="0 0 0"/>
  </joint>
   <joint name="base_to_laser_joint" type="fixed">
     <parent link="base_link"/>
     <child link="base_laser"/>
-    <origin xyz="0.4 0 0.311"/>
+    <origin xyz="0.4 0 0.2297711"/>
   </joint>
   <joint name="base_to_camera1_joint" type="fixed">
@@ -249,3 +250,8 @@
     <origin xyz="-0.3 0 0.6"/>
   </joint>
+  <joint name="imu_joint" type="fixed">
+    <parent link="base_link"/>
+    <child link="imu_link"/>
+    <origin xyz="0.0 0.0 0.2" rpy="0 0 0"/>
+  </joint>
 </robot>

Commit message: add the roll-pitch actuators to stabilize laser on simulation

File: catkin_ws/src/hardware/finder_description/robot/finder_base_8w.gazebo.xacro (robot description, xacro)
@@ -49,4 +49,6 @@
   <xacro:tran joint="right_back_flipper_joint"/>
   <xacro:tran joint="left_back_flipper_joint"/>
+  <xacro:tran joint="laser_roll_joint"/>
+  <xacro:tran joint="laser_pitch_joint"/>
   <gazebo>
     <plugin name="skid_steer_drive_controller" filename="libgazebo_ros_skid_steer_drive.so">

File: catkin_ws/src/hardware/finder_description/robot/finder_base_8w.urdf.xacro (robot description, xacro)
@@ -138,9 +138,37 @@
     </collision>-->
   </link>
+  <link name = "laser_roll">
+    <visual>
+      <origin xyz="0 0 0.0" rpy="0 0 0"/>
+      <geometry>
+        <box size="0.05 0.05 0.05"/>
+      </geometry>
+      <material name="red"/>
+    </visual>
+    <inertial>
+      <mass value="0.100" />
+      <origin xyz="0 0 0" />
+      <inertia ixx="0.001" ixy="0.0" ixz="0.0" iyy="0.001" iyz="0.0" izz="0.001" />
+    </inertial>
+  </link>
+  <link name = "laser_pitch">
+    <visual>
+      <origin xyz="0 0 0.0" rpy="0 0 0"/>
+      <geometry>
+        <box size="0.05 0.05 0.05"/>
+      </geometry>
+      <material name="red"/>
+    </visual>
+    <inertial>
+      <mass value="0.100" />
+      <origin xyz="0 0 0" />
+      <inertia ixx="0.001" ixy="0.0" ixz="0.0" iyy="0.001" iyz="0.0" izz="0.001" />
+    </inertial>
+  </link>
   <link name = "base_laser">
     <visual>
       <origin xyz="0 0 0.0" rpy="0 0 0"/>
       <geometry>
-        <box size="0.01 0.01 0.01"/>
+        <box size="0.05 0.05 0.024"/>
       </geometry>
       <material name="red"/>
@@ -239,9 +267,23 @@
     <child link = "right_belt_link"/>
     <origin xyz="-0.3025 -0.19575 0.0707856" rpy="0 0 0"/>
- </joint>
-  <joint name="base_to_laser_joint" type="fixed">
+  </joint>
+  <joint name="laser_roll_joint" type="revolute">
     <parent link="base_link"/>
+    <child link="laser_roll"/>
+    <origin xyz="0.4 0 0.18"/>
+    <limit lower="-0.5235" upper="0.5235" effort="0.1" velocity="1.57"/>
+    <axis xyz="1 0 0"/>
+  </joint>
+  <joint name="laser_pitch_joint" type="revolute">
+    <parent link="laser_roll"/>
+    <child link="laser_pitch"/>
+    <origin xyz="0.05 0 0.0"/>
+    <limit lower="-0.5235" upper="0.5235" effort="0.1" velocity="1.57"/>
+    <axis xyz="0 1 0"/>
+  </joint>
+  <joint name="pitch_to_laser_joint" type="fixed">
+    <parent link="laser_pitch"/>
     <child link="base_laser"/>
-    <origin xyz="0.4 0 0.2297711"/>
+    <origin xyz="0.0 0 0.0497711"/>
   </joint>
   <joint name="base_to_camera1_joint" type="fixed">
